File: PCB/STAC/STAC.kicad_pcb (KiCad board)
At the start: 2 copper layers, 60.8 x 50.5 mm, 55 parts, among them J1 VIN, J2 BATT, J3 Loadcell, J4 UART, J5 COMM, J6 SW, K1 POWER_SLCT, Q1 MMBT4403, U1 TP4056, U2 SX1308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

Commit message: image update
Parts:
- added JP1: RATE, Jumper:SolderJumper-3_P1.3mm_Bridged12_RoundedPad1.0x1.5mm_NumberLabels, B.Cu at (112.4, 84.5)
Connections:
- U5 pad 15: GND -> Net-(JP1-Pad2)
Routing:
- net Net-(JP1-Pad2): track 0.00 -> 3.75 mm, vias 0 -> 1
- net +5VL: track 109.5 -> 111.6 mm, vias 0 -> 1

Commit message: CIrcuit changed
Parts:
- removed C14, C15: 100nf, Capacitor_SMD:C_0603_1608Metric
- moved C1 57.9 mm to (134.7, 91.7)
- moved C11 57.9 mm to (143.0, 88.8)
- moved C2 57.9 mm to (137.3, 118.9)
- moved C3 57.9 mm to (133.2, 102.6)
- moved C4 57.9 mm to (174.4, 104.5)
- moved C5 57.9 mm to (142.6, 111.3)
- moved C7 57.9 mm to (136.9, 82.5)
- moved D1 57.9 mm to (133.6, 99.2)
- moved D5 57.9 mm to (174.4, 92.3)
- moved D6 57.9 mm to (174.4, 95.6)
- moved J1 57.9 mm to (127.6, 85.7)
- moved J2 57.9 mm to (127.6, 113.9)
- moved J3 57.9 mm to (178.9, 110.7)
- moved J4 57.9 mm to (178.9, 86.6)
- moved J5 57.9 mm to (178.9, 98.7)
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Routing:
- net /IO0: track 37.9 -> 35.8 mm
- net /EN: track 28.4 -> 26.4 mm
Other:
- board text added: "2022.08.25"
- board text added: "V1.2 PNXELEC.COM"
- board text removed: "2022.08.08"
- board text removed: "V1.1 PNXELEC.COM"
