File: PCB/STAC/STAC.sch (KiCad schematic (older format))
At the start: 54 parts, among them J1 VIN, J2 BATT, J3 Loadcell, J4 UART, J5 COMM, J6 SW, K1 POWER_SLCT, Q1 MMBT4403, U1 TP4056, U2 SX1308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

Commit message: image update
Parts:
- added JP1: RATE, Jumper:SolderJumper-3_P1.3mm_Bridged12_RoundedPad1.0x1.5mm_NumberLabels, symbol Jumper:SolderJumper_3_Bridged12
Connections:
- net +5VL: now also JP1.1 (A)
- net GND: now also JP1.3 (B); no longer U5.15 (RATE)
- new net: JP1.2 (C), U5.15 (RATE)
Other:
- moved on the sheet: H1, H3, H4, J4, J5
Changed lines of the file:
@@
 L Connector_Generic:Conn_01x04 J4
 U 1 1 62DEB297
-P 10150 2550
-F 0 "J4" H 10230 2542 50  0000 L CNN
-F 1 "UART" H 10230 2451 50  0000 L CNN
-F 2 "Connector_Molex:Molex_PicoBlade_53261-0471_1x04-1MP_P1.25mm_Horizontal" H 10150 2550 50  0001 C CNN
-F 3 "~" H 10150 2550 50  0001 C CNN
-	1    10150 2550
+P 8550 1550
+F 0 "J4" H 8630 1542 50  0000 L CNN
+F 1 "UART" H 8630 1451 50  0000 L CNN
+F 2 "Connector_Molex:Molex_PicoBlade_53261-0471_1x04-1MP_P1.25mm_Horizontal" H 8550 1550 50  0001 C CNN
+F 3 "~" H 8550 1550 50  0001 C CNN
+	1    8550 1550
 	1    0    0    -1
 $EndComp
@@
 Text Label 7550 1900 0    50   ~ 0
 RX
-Text Label 9950 2550 2    50   ~ 0
+Text Label 8350 1550 2    50   ~ 0
 TX
-Text Label 9950 2450 2    50   ~ 0
+Text Label 8350 1450 2    50   ~ 0
 RX
 $Comp
 L power:GND #PWR0114
 U 1 1 62DF289D
-P 9950 2650
-F 0 "#PWR0114" H 9950 2400 50  0001 C CNN
-F 1 "GND" V 9955 2522 50  0000 R CNN
-F 2 "" H 9950 2650 50  0001 C CNN
-F 3 "" H 9950 2650 50  0001 C CNN
-	1    9950 2650
+P 8350 1650
+F 0 "#PWR0114" H 8350 1400 50  0001 C CNN
+F 1 "GND" V 8355 1522 50  0000 R CNN
+F 2 "" H 8350 1650 50  0001 C CNN
+F 3 "" H 8350 1650 50  0001 C CNN
+	1    8350 1650
 	0    1    1    0
 $EndComp
@@
 L power:+5VL #PWR0135
 U 1 1 62DA431F
-P 9950 2750
-F 0 "#PWR0135" H 9950 2600 50  0001 C CNN
-F 1 "+5VL" V 9965 2878 50  0000 L CNN
-F 2 "" H 9950 2750 50  0001 C CNN
-F 3 "" H 9950 2750 50  0001 C CNN
-	1    9950 2750
+P 8350 1750
+F 0 "#PWR0135" H 8350 1600 50  0001 C CNN
+F 1 "+5VL" V 8365 1878 50  0000 L CNN
+F 2 "" H 8350 1750 50  0001 C CNN
+F 3 "" H 8350 1750 50  0001 C CNN
+	1    8350 1750
 	0    -1   -1   0
 $EndComp
@@
 L power:GND #PWR0140
 U 1 1 62EDF9BA
-P 7500 5150
-F 0 "#PWR0140" H 7500 4900 50  0001 C CNN
-F 1 "GND" V 7505 5022 50  0000 R CNN
-F 2 "" H 7500 5150 50  0001 C CNN
-F 3 "" H 7500 5150 50  0001 C CNN
-	1    7500 5150
-	0    -1   -1   0
+P 8150 5350
+F 0 "#PWR0140" H 8150 5100 50  0001 C CNN
+F 1 "GND" V 8155 5222 50  0000 R CNN
+F 2 "" H 8150 5350 50  0001 C CNN
+F 3 "" H 8150 5350 50  0001 C CNN
+	1    8150 5350
+	1    0    0    -1
 $EndComp
 $Comp
@@
 L Connector_Generic:Conn_01x04 J5
 U 1 1 62FDB005
-P 10150 3050
-F 0 "J5" H 10230 3042 50  0000 L CNN
-F 1 "COMM" H 10230 2951 50  0000 L CNN
-F 2 "Connector_Molex:Molex_PicoBlade_53261-0471_1x04-1MP_P1.25mm_Horizontal" H 10150 3050 50  0001 C CNN
-F 3 "~" H 10150 3050 50  0001 C CNN
-	1    10150 3050
+P 8550 2050
+F 0 "J5" H 8630 2042 50  0000 L CNN
+F 1 "COMM" H 8630 1951 50  0000 L CNN
+F 2 "Connector_Molex:Molex_PicoBlade_53261-0471_1x04-1MP_P1.25mm_Horizontal" H 8550 2050 50  0001 C CNN
+F 3 "~" H 8550 2050 50  0001 C CNN
+	1    8550 2050
 	1    0    0    -1
 $EndComp
@@
 L power:+5VL #PWR0149
 U 1 1 62FE7338
-P 9950 3250
-F 0 "#PWR0149" H 9950 3100 50  0001 C CNN
-F 1 "+5VL" V 9965 3377 50  0000 L CNN
-F 2 "" H 9950 3250 50  0001 C CNN
-F 3 "" H 9950 3250 50  0001 C CNN
-	1    9950 3250
+P 8350 2250
+F 0 "#PWR0149" H 8350 2100 50  0001 C CNN
+F 1 "+5VL" V 8365 2377 50  0000 L CNN
+F 2 "" H 8350 2250 50  0001 C CNN
+F 3 "" H 8350 2250 50  0001 C CNN
+	1    8350 2250
 	0    -1   -1   0
 $EndComp
@@
 L power:GND #PWR0150
 U 1 1 62FE7AAD
-P 9950 3150
-F 0 "#PWR0150" H 9950 2900 50  0001 C CNN
-F 1 "GND" V 9955 3022 50  0000 R CNN
-F 2 "" H 9950 3150 50  0001 C CNN
-F 3 "" H 9950 3150 50  0001 C CNN
-	1    9950 3150
+P 8350 2150
+F 0 "#PWR0150" H 8350 1900 50  0001 C CNN
+F 1 "GND" V 8355 2022 50  0000 R CNN
+F 2 "" H 8350 2150 50  0001 C CNN
+F 3 "" H 8350 2150 50  0001 C CNN
+	1    8350 2150
 	0    1    1    0
 $EndComp
-Text Label 9950 2950 2    50   ~ 0
+Text Label 8350 1950 2    50   ~ 0
 RX_COMM
-Text Label 9950 3050 2    50   ~ 0
+Text Label 8350 2050 2    50   ~ 0
 TX_COMM
 $Comp
@@
 L Mechanical:MountingHole H1
 U 1 1 62E145BD
-P 9900 5400
-F 0 "H1" H 10000 5446 50  0000 L CNN
-F 1 "MountingHole" H 10000 5355 50  0000 L CNN
-F 2 "MountingHole:MountingHole_3.2mm_M3" H 9900 5400 50  0001 C CNN
-F 3 "~" H 9900 5400 50  0001 C CNN
-	1    9900 5400
+P 10050 5500
+F 0 "H1" H 10150 5546 50  0000 L CNN
+F 1 "MountingHole" H 10150 5455 50  0000 L CNN
+F 2 "MountingHole:MountingHole_3.2mm_M3" H 10050 5500 50  0001 C CNN
+F 3 "~" H 10050 5500 50  0001 C CNN
+	1    10050 5500
 	1    0    0    -1
 $EndComp
@@
 L Mechanical:MountingHole H3
 U 1 1 62E15224
-P 10550 5200
-F 0 "H3" H 10650 5246 50  0000 L CNN
-F 1 "MountingHole" H 10650 5155 50  0000 L CNN
-F 2 "MountingHole:MountingHole_3.2mm_M3" H 10550 5200 50  0001 C CNN
-F 3 "~" H 10550 5200 50  0001 C CNN
-	1    10550 5200
+P 10050 6000
+F 0 "H3" H 10150 6046 50  0000 L CNN
+F 1 "MountingHole" H 10150 5955 50  0000 L CNN
+F 2 "MountingHole:MountingHole_3.2mm_M3" H 10050 6000 50  0001 C CNN
+F 3 "~" H 10050 6000 50  0001 C CNN
+	1    10050 6000
 	1    0    0    -1
 $EndComp
@@
 L Mechanical:MountingHole H4
 U 1 1 62E15E41
-P 10600 5800
-F 0 "H4" H 10700 5846 50  0000 L CNN
-F 1 "MountingHole" H 10700 5755 50  0000 L CNN
-F 2 "MountingHole:MountingHole_3.2mm_M3" H 10600 5800 50  0001 C CNN
-F 3 "~" H 10600 5800 50  0001 C CNN
-	1    10600 5800
+P 10050 6250
+F 0 "H4" H 10150 6296 50  0000 L CNN
+F 1 "MountingHole" H 10150 6205 50  0000 L CNN
+F 2 "MountingHole:MountingHole_3.2mm_M3" H 10050 6250 50  0001 C CNN
+F 3 "~" H 10050 6250 50  0001 C CNN
+	1    10050 6250
 	1    0    0    -1
 $EndComp
@@
 	0    -1   -1   0
 $EndComp
+Wire Wire Line
+	7500 5150 8000 5150
+$Comp
+L power:+5VL #PWR0157
+U 1 1 62F53F6C
+P 8150 4950
+F 0 "#PWR0157" H 8150 4800 50  0001 C CNN
+F 1 "+5VL" H 8165 5123 50  0000 C CNN
+F 2 "" H 8150 4950 50  0001 C CNN
+F 3 "" H 8150 4950 50  0001 C CNN
+	1    8150 4950
+	1    0    0    -1
+$EndComp
+$Comp
+L Jumper:SolderJumper_3_Bridged12 JP1
+U 1 1 62F5DA7B
+P 8150 5150
+F 0 "JP1" V 8104 5218 50  0000 L CNN
+F 1 "RATE" V 8195 5218 50  0000 L CNN
+F 2 "Jumper:SolderJumper-3_P1.3mm_Bridged12_RoundedPad1.0x1.5mm_NumberLabels" H 8150 5150 50  0001 C CNN
+F 3 "~" H 8150 5150 50  0001 C CNN
+	1    8150 5150
+	0    1    1    0
+$EndComp
 $EndSCHEMATC

Commit message: CIrcuit changed
Parts:
- removed C14, C15: 100nf, Capacitor_SMD:C_0603_1608Metric, symbol Device:C_Small
Changed lines of the file:
@@
-$EndComp
-$Comp
-L Device:C_Small C15
-U 1 1 62F4B28D
-P 5750 3800
-F 0 "C15" H 5842 3846 50  0000 L CNN
-F 1 "100nf" H 5842 3755 50  0000 L CNN
-F 2 "Capacitor_SMD:C_0603_1608Metric" H 5750 3800 50  0001 C CNN
-F 3 "~" H 5750 3800 50  0001 C CNN
-	1    5750 3800
-	1    0    0    -1
-$EndComp
-$Comp
-L power:GND #PWR0153
-U 1 1 62F4B293
-P 5750 3900
-F 0 "#PWR0153" H 5750 3650 50  0001 C CNN
-F 1 "GND" H 5755 3727 50  0000 C CNN
-F 2 "" H 5750 3900 50  0001 C CNN
-F 3 "" H 5750 3900 50  0001 C CNN
-	1    5750 3900
-	1    0    0    -1
-$EndComp
-$Comp
-L Device:C_Small C14
-U 1 1 62F64D96
-P 5750 3250
-F 0 "C14" H 5842 3296 50  0000 L CNN
-F 1 "100nf" H 5842 3205 50  0000 L CNN
-F 2 "Capacitor_SMD:C_0603_1608Metric" H 5750 3250 50  0001 C CNN
-F 3 "~" H 5750 3250 50  0001 C CNN
-	1    5750 3250
-	1    0    0    -1
-$EndComp
-$Comp
-L power:GND #PWR0154
-U 1 1 62F64D9C
-P 5750 3350
-F 0 "#PWR0154" H 5750 3100 50  0001 C CNN
-F 1 "GND" H 5755 3177 50  0000 C CNN
-F 2 "" H 5750 3350 50  0001 C CNN
-F 3 "" H 5750 3350 50  0001 C CNN
-	1    5750 3350
-	1    0    0    -1
 $EndComp
 $Comp
